File: PCB/harp timestamp generator Gen3.sch (EAGLE design)
At the start: 140 parts, among them IC1 SI8621BC-B-IS, IC10 SN74LVC1G125DBVT, IC11 SI8621BC-B-IS, IC12 SI8621BC-B-IS, IC13 SI8621BC-B-IS, IC14 SI8621BC-B-IS, IC15 ATXMEGAxxxA4U-AU, IC16 74AHC1G126DCK, IC18 74AHC1G126DCK, IC2 USBLC6-2SC6, IC3 FT232RL, IC4 TLV70033DDCR, IC5 TLV70033DDCR, IC6 SI8621BC-B-IS, IC7 74AHC1G126DCK, IC8 SN74LVC1G125DBVT, IC9 SN74LVC1G125DBVT, Q1 RTU002P02T106, Q2 BC817-40W, Q3 BC817-40LT1SMD, Q6 DMP2035U-7, T10 BC850, T11 BC850, T12 BC850, T13 BC850, T4 BC850, T5 BC850, T6 BC850, T7 BC850, T8 BC850, T9 BC850, U1 MCP73831T-2ATI/OT, U2 ICL7673CBAZA-T, X1 B2B-PH-K-S(LF)(SN)

Commit message: Corrected buffers' enable.
Parts:
- removed T11, T12, T13: BC850, transistor:BC850
- removed U1: MCP73831T-2ATI/OT, harp timestamp generator:MCP73831T-2ATI/OT
- removed U2: ICL7673CBAZA-T, harp timestamp generator:ICL7673CBAZA-T
- added IC17: SI8621BC-B-IS, harp timestamp generator:SI8621BC-B-IS
- added IC19: SN74LVC1G125DBVT, 74xx-little-de:74AHC1G125DBV
- added T1, T2, T3: BC850, transistor:BC850
- IC1: value SI8621BC-B-IS -> MCP73831T-2ATI/OT; device harp timestamp generator:SI8621BC-B-IS -> harp timestamp generator:MCP73831T-2ATI/OT; MPN Si8621BC-B-IS -> MCP73831T-2ATI/OT
- IC11: value SI8621BC-B-IS -> TLV70033DDCR; device harp timestamp generator:SI8621BC-B-IS -> harp timestamp generator:TLV700XX; MPN Si8621BC-B-IS -> TLV70033DDCR
- IC15: value ATXMEGAxxxA4U-AU -> SI8621BC-B-IS; device harp timestamp generator:AT-XMEGA-XXA4-AU -> harp timestamp generator:SI8621BC-B-IS; MPN (none) -> Si8621BC-B-IS
- IC16: value 74AHC1G126DCK -> SI8621BC-B-IS; device 74xx-little-de:74AHC1G126DCK -> harp timestamp generator:SI8621BC-B-IS; MPN (none) -> Si8621BC-B-IS
- IC18: value 74AHC1G126DCK -> SN74LVC1G125DBVT; device 74xx-little-de:74AHC1G126DCK -> 74xx-little-de:74AHC1G125DBV; MPN (none) -> SN74LVC1G125DBVT
- IC4: value TLV70033DDCR -> ICL7673CBAZA-T; device harp timestamp generator:TLV700XX -> harp timestamp generator:ICL7673CBAZA-T; MPN TLV70033DDCR -> (none)
- IC6: value SI8621BC-B-IS -> ATXMEGAxxxA4U-AU; device harp timestamp generator:SI8621BC-B-IS -> harp timestamp generator:AT-XMEGA-XXA4-AU; MPN Si8621BC-B-IS -> (none)
- IC7: value 74AHC1G126DCK -> M74VHC1GT126DF1G
- IC8, IC9: value SN74LVC1G125DBVT -> M74VHC1GT126DF1G; device 74xx-little-de:74AHC1G125DBV -> 74xx-little-de:74AHC1G126DCK; MPN SN74LVC1G125DBVT -> (none)
- renumbered Q6 to Q5, TEST to BUTTON
Connections:
- net +3V3: now also IC15.AVDD, IC16.AVDD, IC17.AVDD, IC18P.VCC, IC19P.VCC, IC5.OUT; no longer IC1.AVDD, IC11.AVDD, IC4.OUT, IC6.AVDD, IC8P.VCC, IC9P.VCC
- net +5V: now also IC11.EN, IC11.IN, IC4.VO, IC7A.OE, IC8A.OE, IC8P.VCC, IC9A.OE, IC9P.VCC; no longer IC16P.VCC, IC18P.VCC, IC4.EN, IC4.IN, U2.VO
- net +5_USB: now also IC4.VP; no longer U2.VP
- net BAT_READ: now also IC6.PA1/ADC1; no longer IC15.PA1/ADC1
- net BAT_VOLTAGE: now also IC6.PA0/ADC0/AREF; no longer IC15.PA0/ADC0/AREF
- net BLIGHT_EN_UC: now also IC6.PA5/ADC5, IC8A.I; no longer IC15.PA5/ADC5, IC16A.I
- net BUTTON: now also IC6.PB3/ADC11/DAC1; no longer IC15.PB3/ADC11/DAC1
- net CHARGE_ENABLE: now also IC6.PB1/ADC9; no longer IC15.PB1/ADC9
- net CLKOUT0: now also IC12.B1_OUT; no longer IC6.B1_OUT
- net CLKOUT1: now also IC13.B1_OUT; no longer IC1.B1_OUT
- net CLKOUT2: now also IC14.B1_OUT; no longer IC11.B1_OUT
- net CLKOUT3: now also IC15.B1_OUT; no longer IC12.B1_OUT
- net CLKOUT4: now also IC16.B1_OUT; no longer IC13.B1_OUT
- net CLKOUT5: now also IC17.B1_OUT; no longer IC14.B1_OUT
- net CLOCK_IN: now also IC18A.I, IC6.!!RXD1MISOPD6; no longer IC15.!!RXD1MISOPD6, IC8A.I
- net CLOCK_OUT: now also IC19A.I, IC6.!!!TXD1SCKCLKOPD7; no longer IC15.!!!TXD1SCKCLKOPD7, IC9A.I
- net CLOCK_OUT_ISO: now also IC15.A1_IN, IC16.A1_IN, IC17.A1_IN, IC18A.O, IC19A.O; no longer IC1.A1_IN, IC11.A1_IN, IC6.A1_IN, IC8A.O, IC9A.O
- net DEVICE_AT_0: now also IC12.A2_OUT, IC6.PC6/MISO/RXD1; no longer IC15.PC6/MISO/RXD1, IC6.A2_OUT
- net DEVICE_AT_1: now also IC13.A2_OUT, IC6.PC7/SCK/TXD1/CLKO/EVO; no longer IC1.A2_OUT, IC15.PC7/SCK/TXD1/CLKO/EVO
- net DEVICE_AT_2: now also IC14.A2_OUT, IC6.PA4/ADC4; no longer IC11.A2_OUT, IC15.PA4/ADC4
- net DEVICE_AT_3: now also IC15.A2_OUT, IC6.PR0/XTAL2; no longer IC12.A2_OUT, IC15.PR0/XTAL2
- net DEVICE_AT_4: now also IC16.A2_OUT, IC6.PA2/ADC2; no longer IC13.A2_OUT, IC15.PA2/ADC2
- net DEVICE_AT_5: now also IC17.A2_OUT, IC6.PA3/ADC3; no longer IC14.A2_OUT, IC15.PA3/ADC3
- net DISCHARGE_BAT: now also IC6.PB2/ADC10/DAC0; no longer IC15.PB2/ADC10/DAC0
- net EN_CLOCK_IN: now also IC18A.OE, IC6.!!OC0CRXD0PD2; no longer IC15.!!OC0CRXD0PD2, IC8A.OE
- net EN_CLOCK_OUT: now also IC19A.OE, IC6.!!OC0BXCK0PD1; no longer IC15.!!OC0BXCK0PD1, IC9A.OE
- net FTDI_CTS: now also IC6.!!XCK0OC0BSCLPE1; no longer IC15.!!XCK0OC0BSCLPE1
- net FTDI_RTS: now also IC6.!OC0ASDAPE0; no longer IC15.!OC0ASDAPE0
- net FTDI_RXD: now also IC6.!!TXD0OC0DPE3; no longer IC15.!!TXD0OC0DPE3
- net FTDI_TXD: now also IC6.!!RXD0OC0CPE2; no longer IC15.!!RXD0OC0CPE2
- net GND: now also IC1.VSS, IC11.GND, IC15.AGND, IC16.AGND, IC17.AGND, IC19P.GND, IC6.GND@1, IC6.GND@2, IC6.GND@3, IC6.GND@4, T1.E, T2.E, T3.E; no longer IC1.AGND, IC11.AGND, IC15.GND@1, IC15.GND@2, IC15.GND@3, IC15.GND@4, IC16P.GND, IC6.AGND, T11.E, T12.E, T13.E, U1.VSS, U2.GND
- net GND_ISO: now also IC12.BGND; no longer IC6.BGND
- net GND_ISO1: now also IC13.BGND; no longer IC1.BGND
- net GND_ISO2: now also IC14.BGND; no longer IC11.BGND
- net GND_ISO3: now also IC15.BGND; no longer IC12.BGND
- net GND_ISO4: now also IC16.BGND; no longer IC13.BGND
- net GND_ISO5: now also IC17.BGND; no longer IC14.BGND
- net LED_CLK_0: now also IC6.PC0/OC0A/SDA; no longer IC15.PC0/OC0A/SDA
- net LED_CLK_1: now also IC6.PC1/OC0B/XCK0/SCL; no longer IC15.PC1/OC0B/XCK0/SCL
- net LED_CLK_2: now also IC6.PC2/OC0C/RXD0; no longer IC15.PC2/OC0C/RXD0
- net LED_CLK_3: now also IC6.PC3/OC0D/TXD0; no longer IC15.PC3/OC0D/TXD0
- net LED_CLK_4: now also IC6.PC4/OC1A/#SS; no longer IC15.PC4/OC1A/#SS
- net LED_CLK_5: now also IC6.PC5/OC1B/MOSI/XCK1; no longer IC15.PC5/OC1B/MOSI/XCK1
- net LED_LOCK: now also IC6.!#SSPD4; no longer IC15.!#SSPD4
- net LED_PWR: now also IC6.!OC0APD0; no longer IC15.!OC0APD0
- net LED_REP: now also IC6.!!OC0DTXD0PD3; no longer IC15.!!OC0DTXD0PD3
- net N$1: now also T7.B; no longer T10.B
- net N$10: now also IC1.VDD; no longer U1.VDD
- net N$11: now also IC14.B2_IN, IC14.BVDD; no longer IC11.B2_IN, IC11.BVDD
- net N$15: now also T3.B; no longer T6.B
- net N$16: now also IC1.PROG; no longer U1.PROG
- net N$17: now also T1.B; no longer T4.B
- net N$19: now also T1.C; no longer T4.C
- net N$20: now also T2.B; no longer T5.B
- net N$21: now also T3.C; no longer T6.C
- net N$22: now also T2.C; no longer T5.C
- net N$24: now also T4.B; no longer T7.B
- net N$25: now also T4.C; no longer T7.C
- net N$26: now also T5.B; no longer T8.B
- net N$27: now also T5.C; no longer T8.C
- net N$28: now also T6.B; no longer T9.B
- net N$29: now also T6.C; no longer T9.C
- net N$3: now also IC8A.O; no longer IC16A.O
- net N$34: now also T8.B; no longer T11.B
- net N$37: now also IC15.B2_IN, IC15.BVDD; no longer IC12.B2_IN, IC12.BVDD
- net N$4: now also IC9A.O; no longer IC18A.O
- net N$42: now also IC11.OUT; no longer IC5.OUT
- net N$45: now also IC16.B2_IN, IC16.BVDD; no longer IC13.B2_IN, IC13.BVDD
- net N$47: now also T8.C; no longer T11.C
- net N$49: now also IC17.B2_IN, IC17.BVDD; no longer IC14.B2_IN, IC14.BVDD
- net N$5: now also IC12.B2_IN, IC12.BVDD; no longer IC6.B2_IN, IC6.BVDD
- net N$53: now also T9.B; no longer T12.B
- net N$54: now also T9.C; no longer T12.C
- net N$56: now also T10.B; no longer T13.B
- net N$6: now also IC13.B2_IN, IC13.BVDD; no longer IC1.B2_IN, IC1.BVDD
- net N$60: now also T10.C; no longer T13.C
- net N$7: now also T7.C; no longer T10.C
- net N$97: now also IC1.VBAT; no longer U1.VBAT
- net OSC1: now also IC6.PR1/XTAL1; no longer IC15.PR1/XTAL1
- net PDI-CLK: now also IC6.RESET/PDI-CLK; no longer IC15.RESET/PDI-CLK
- net PDI-DATA: now also IC6.PDI-DATA; no longer IC15.PDI-DATA
- net PWR_GOOD: now also IC4.P_BAR, IC6.PB0/ADC8/AREF; no longer IC15.PB0/ADC8/AREF, U2.P_BAR
- net STATE: now also IC6.!!XCK1MOSIPD5; no longer IC15.!!XCK1MOSIPD5
- net UC_RX: now also IC6.PA6/ADC6; no longer IC15.PA6/ADC6
- net UC_TX: now also IC6.PA7/ADC7/AC0-OUT, IC9A.I; no longer IC15.PA7/ADC7/AC0-OUT, IC18A.I
- net VDD: now also IC6.AVCC, IC6.VCC@1, IC6.VCC@2, IC6.VCC@3; no longer IC15.AVCC, IC15.VCC@1, IC15.VCC@2, IC15.VCC@3
- net V_BATT: now also IC4.VS; no longer U2.VS
Other:
- moved on the sheet: IC12, IC13, IC14, IC18, IC18P, IC5, IC7, IC8, IC8P, IC9, IC9P, T10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

Commit message: Big updates. Very close to final design.
Parts:
- BUTTON: DIGKEYPN (none) -> 563-1246-1-ND; MPN (none) -> CFPA-1FB4-A2T
- C1, C12, C13, C14, C15, C16, C17, C18, C19, C20, C21, C25, C26, C3, C30, C31, C35, C36, C37, C38, C5, C7, C9: DIGKEYPN (none) -> 445-6899-2-ND; MPN MC0402B104K160CT -> CGA2B3X7R1H104K050BB
- C10, C11, C23, C24: DIGKEYPN (none) -> 541-10.0YCT-ND; MPN C1608X6S1C475K080AC -> CRCW040210R0FKEDHP
- C2: DIGKEYPN (none) -> 587-2237-1-ND; MPN 885012205084 -> UMK105B7472KV-F
- C22, C27, C28, C29, C32, C62: DIGKEYPN (none) -> 445-6899-2-ND; MPN (none) -> CGA2B3X7R1H104K050BB
- C33: value 4.7n -> 10n; DIGKEYPN (none) -> 1276-1028-1-ND; MPN ?? -> CL05B103KB5NNNC
- C34: DIGKEYPN (none) -> 1276-1028-1-ND; MPN ?? -> CL05B103KB5NNNC
- C4, C6: DIGKEYPN (none) -> 478-1171-1-ND; MPN 04025A470JAT2A -> 06035A470JAT2A
- C8: DIGKEYPN (none) -> 478-11183-1-ND; MPN TAJA475K016UNJ -> TAJA475K010TNJ
- CLKIN, CLKOUT0, CLKOUT1, CLKOUT2, CLKOUT3, CLKOUT4, CLKOUT5: DIGKEYPN (none) -> SC1489-1-ND
- F1: value 10MHz ?? -> 330 Ohms @ 100MHz; DIGKEYPN (none) -> 490-3997-1-ND; MPN (none) -> BLM18SG331TN1D
- IC1: DIGKEYPN (none) -> MCP73831T-2ATI/OTCT-ND; MPN MCP73831T-2ATI/OT -> (none)
- IC10, IC18, IC19: DIGKEYPN (none) -> 296-26595-1-ND
- IC11, IC5: DIGKEYPN (none) -> 296-27937-6-ND
- IC12, IC13, IC14, IC15, IC16, IC17: DIGKEYPN (none) -> 336-2064-5-ND
- IC2: DIGKEYPN (none) -> 497-5235-1-ND
- IC3: DIGKEYPN (none) -> 768-1007-1-ND
- IC4: DIGKEYPN (none) -> ICL7673CBAZA-TCT-ND; MPN (none) -> ICL7673CBAZA-T
- IC6: value ATXMEGAxxxA4U-AU -> ATXMEGA16A4U-AU; DIGKEYPN (none) -> ATXMEGA16A4U-AU-ND; MPN (none) -> ATXMEGA16A4U-AU
- IC7, IC8, IC9: DIGKEYPN (none) -> M74VHC1GT126DF1GOSCT-ND; MPN (none) -> M74VHC1GT126DF1G
- L1: DIGKEYPN (none) -> 240-2389-1-ND
- LED1, LED2, LED3, LED4, LED5: DIGKEYPN (none) -> 350-1782-ND
- OSC1: DIGKEYPN (none) -> 1908-1044-1-ND; MPN (none) -> O 32,0-JT32C-A-K-3,3-LF
- PDI: value (none) -> 2x3_header; DIGKEYPN (none) -> 609-3210-ND; MPN (none) -> 67996-206HLF
- Q1: DIGKEYPN (none) -> RTU002P02T106CT-ND; MPN (none) -> RTU002P02T106
- Q2: DIGKEYPN (none) -> 1727-6185-1-ND; MPN (none) -> BC817-40W,135
- Q3: DIGKEYPN (none) -> SBC817-40LT1GOSCT-ND; MPN (none) -> SBC817-40LT1G
- Q4: value (none) -> DMG1012UW; DIGKEYPN (none) -> DMG1012UW-7DICT-ND; MPN (none) -> DMG1012UW-7
- Q5: DIGKEYPN (none) -> DMP2035U-7DICT-ND
- R1: DIGKEYPN (none) -> 541-3965-1-ND; MPN CRCW04021M00FKED -> CRCW04021M00FKEDC
- R10, R11, R12: DIGKEYPN (none) -> 311-100DCT-ND; MPN CRCW0603100RFKEAHP -> RT0603DRD07100RL
- R13, R17, R19: DIGKEYPN (none) -> YAG1444CT-ND; MPN 22k !!! -> RT0402BRD074K53L
- R14: value 10k ?? -> 10k; DIGKEYPN (none) -> 541-3959-1-ND; MPN ??? -> CRCW040210K0FKEDC
- R15: DIGKEYPN (none) -> 541-2662-1-ND; MPN ??? -> RCP2512W25R0GEB
- R16, R18, R3, R7: DIGKEYPN (none) -> 541-3959-1-ND; MPN CRCW040210K0FKED -> CRCW040210K0FKEDC
- R2: DIGKEYPN (none) -> 541-10.0YCT-ND
- R21, R22, R23, R24, R25, R27, R28, R29, R30, R31: DIGKEYPN (none) -> 541-1.00KYCT-ND
- R33, R34, R35, R36, R37, R40, R41, R42, R44, R45: DIGKEYPN (none) -> 311-330LRCT-ND
- R4: DIGKEYPN (none) -> P51KDCCT-ND; MPN CRCW040210K0FKED -> ERA-2AEB513X
- R48: DIGKEYPN (none) -> 311-100KHRCT-ND; MPN (none) -> RC0603FR-07100KL
- R5: value 15K 0.1% -> 15K 0.1% => 14k7; DIGKEYPN (none) -> YAG4174CT-ND; MPN CRCW040210K0FKED -> RT0402BRD0714K7L
- R54, R55: DIGKEYPN (none) -> 541-3959-1-ND
- R6: DIGKEYPN (none) -> 311-100KHRCT-ND; MPN CRCW040210K0FKED -> RC0603FR-07100KL
- R8: DIGKEYPN (none) -> 311-0.0HRCT-ND; MPN CRCW040210K0FKED -> RC0603FR-070RL
- R9: DIGKEYPN (none) -> 541-3959-1-ND; MPN (none) -> CRCW040210K0FKEDC
- SV1: DIGKEYPN (none) -> S9177-ND
- T1, T10, T2, T3, T4, T5, T6, T7, T8, T9: DIGKEYPN (none) -> 1727-4862-1-ND
- USB: DIGKEYPN (none) -> H2960TR-ND; MPN UX60-MB-5S8 -> UX60-MB-5S8
- X1: DIGKEYPN (none) -> 455-1704-ND; MPN (none) -> B2B-PH-K-S(LF)(SN)

Commit message: Increased battery current draw to around 250 mA.
Parts:
- R15: value 25R -> 15R
Changed lines of the file:
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@@
 <?xml version="1.0" encoding="utf-8"?>
 <!DOCTYPE eagle SYSTEM "eagle.dtd">
-<eagle version="9.6.2">
+<eagle version="9.5.1">
 <drawing>
 <settings>
@@
 <attribute name="MPN" value="CRCW040210K0FKEDC"/>
 </part>
-<part name="R15" library="rcl" deviceset="R-EU_" device="R2512" value="25R">
+<part name="R15" library="rcl" deviceset="R-EU_" device="R2512" value="15R">
 <attribute name="DIGKEYPN" value="541-2662-1-ND"/>
 <attribute name="MPN" value="RCP2512W25R0GEB"/>

Commit message: Updated files with the MPN.
Parts:
- C10, C11, C23, C24: DIGKEYPN 541-10.0YCT-ND -> 587-2786-1-ND; MPN CRCW040210R0FKEDHP -> EMK107ABJ475KA-T
- C29: DIGKEYPN 445-6899-2-ND -> 490-3263-1-ND; MPN CGA2B3X7R1H104K050BB -> GRM155R61A334KE15D
- C4, C6: DIGKEYPN 478-1171-1-ND -> 478-1078-1-ND; MPN 06035A470JAT2A -> 04025A470JAT2A
- R21, R22, R23, R24, R25, R27, R28, R29, R30, R31: MPN CRCW04021K00FKED -> CRCW04021K00FKEDHP
- R48, R6: DIGKEYPN 311-100KHRCT-ND -> P15984CT-ND; MPN RC0603FR-07100KL -> ERJ-2RHD1002X
- R54, R55: DIGKEYPN 541-3959-1-ND -> 541-1.00KYCT-ND; MPN CRCW040210K0FKED -> CRCW04021K00FKEDHP
- R8: DIGKEYPN 311-0.0HRCT-ND -> RMCF0402ZT0R00CT-ND; MPN RC0603FR-070RL -> RMCF0402ZT0R00
Changed lines of the file:
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@@
 <?xml version="1.0" encoding="utf-8"?>
 <!DOCTYPE eagle SYSTEM "eagle.dtd">
-<eagle version="9.5.1">
+<eagle version="9.6.2">
 <drawing>
 <settings>
@@
 </part>
 <part name="C4" library="rcl" deviceset="C-EU" device="C0402" value="47pF">
-<attribute name="DIGKEYPN" value="478-1171-1-ND"/>
-<attribute name="MPN" value="06035A470JAT2A"/>
+<attribute name="DIGKEYPN" value="478-1078-1-ND"/>
+<attribute name="MPN" value="04025A470JAT2A"/>
 </part>
 <part name="C6" library="rcl" deviceset="C-EU" device="C0402" value="47pF">
-<attribute name="DIGKEYPN" value="478-1171-1-ND"/>
-<attribute name="MPN" value="06035A470JAT2A"/>
+<attribute name="DIGKEYPN" value="478-1078-1-ND"/>
+<attribute name="MPN" value="04025A470JAT2A"/>
 </part>
 <part name="L1" library="rcl" deviceset="R-EU_" device="R0805" value="40R@100MHz">
@@
 <part name="R21" library="rcl" deviceset="R-EU_" device="R0402" value="1k">
 <attribute name="DIGKEYPN" value="541-1.00KYCT-ND"/>
-<attribute name="MPN" value="CRCW04021K00FKED"/>
+<attribute name="MPN" value="CRCW04021K00FKEDHP"/>
 </part>
 <part name="R33" library="rcl" deviceset="R-EU_" device="R0402" value="330R">
@@
 <part name="R27" library="rcl" deviceset="R-EU_" device="R0402" value="1k">
 <attribute name="DIGKEYPN" value="541-1.00KYCT-ND"/>
-<attribute name="MPN" value="CRCW04021K00FKED"/>
+<attribute name="MPN" value="CRCW04021K00FKEDHP"/>
 </part>
 <part name="R40" library="rcl" deviceset="R-EU_" device="R0402" value="330R">
@@
 <part name="R22" library="rcl" deviceset="R-EU_" device="R0402" value="1k">
 <attribute name="DIGKEYPN" value="541-1.00KYCT-ND"/>
-<attribute name="MPN" value="CRCW04021K00FKED"/>
+<attribute name="MPN" value="CRCW04021K00FKEDHP"/>
 </part>
 <part name="R34" library="rcl" deviceset="R-EU_" device="R0402" value="330R">
@@
 <part name="R28" library="rcl" deviceset="R-EU_" device="R0402" value="1k">
 <attribute name="DIGKEYPN" value="541-1.00KYCT-ND"/>
-<attribute name="MPN" value="CRCW04021K00FKED"/>
+<attribute name="MPN" value="CRCW04021K00FKEDHP"/>
 </part>
 <part name="R41" library="rcl" deviceset="R-EU_" device="R0402" value="330R">
@@
 <part name="R23" library="rcl" deviceset="R-EU_" device="R0402" value="1k">
 <attribute name="DIGKEYPN" value="541-1.00KYCT-ND"/>
-<attribute name="MPN" value="CRCW04021K00FKED"/>
+<attribute name="MPN" value="CRCW04021K00FKEDHP"/>
 </part>
 <part name="R35" library="rcl" deviceset="R-EU_" device="R0402" value="330R">
@@
 <part name="R29" library="rcl" deviceset="R-EU_" device="R0402" value="1k">
 <attribute name="DIGKEYPN" value="541-1.00KYCT-ND"/>
-<attribute name="MPN" value="CRCW04021K00FKED"/>
+<attribute name="MPN" value="CRCW04021K00FKEDHP"/>
 </part>
 <part name="R42" library="rcl" deviceset="R-EU_" device="R0402" value="330R">
@@
 </part>
 <part name="C24" library="rcl" deviceset="C-EU" device="C0603" value="4.7uF">
-<attribute name="DIGKEYPN" value="541-10.0YCT-ND"/>
-<attribute name="MPN" value="CRCW040210R0FKEDHP"/>
+<attribute name="DIGKEYPN" value="587-2786-1-ND"/>
+<attribute name="MPN" value="EMK107ABJ475KA-T"/>
 </part>
 <part name="IC11" library="harp timestamp generator" deviceset="TLV700XX" device="" value="TLV70033DDCR">
@@
 </part>
 <part name="C23" library="rcl" deviceset="C-EU" device="C0603" value="4.7uF">
-<attribute name="DIGKEYPN" value="541-10.0YCT-ND"/>
-<attribute name="MPN" value="CRCW040210R0FKEDHP"/>
+<attribute name="DIGKEYPN" value="587-2786-1-ND"/>
+<attribute name="MPN" value="EMK107ABJ475KA-T"/>
 </part>
 <part name="GND57" library="supply1" deviceset="GND" device="">
@@
 <part name="GND86" library="supply1" deviceset="GND" device=""/>
 <part name="C11" library="rcl" deviceset="C-EU" device="C0603" value="4.7uF">
-<attribute name="DIGKEYPN" value="541-10.0YCT-ND"/>
-<attribute name="MPN" value="CRCW040210R0FKEDHP"/>
+<attribute name="DIGKEYPN" value="587-2786-1-ND"/>
+<attribute name="MPN" value="EMK107ABJ475KA-T"/>
 </part>
 <part name="IC5" library="harp timestamp generator" deviceset="TLV700XX" device="" value="TLV70033DDCR">
@@
 </part>
 <part name="C10" library="rcl" deviceset="C-EU" device="C0603" value="4.7uF">
-<attribute name="DIGKEYPN" value="541-10.0YCT-ND"/>
-<attribute name="MPN" value="CRCW040210R0FKEDHP"/>
+<attribute name="DIGKEYPN" value="587-2786-1-ND"/>
+<attribute name="MPN" value="EMK107ABJ475KA-T"/>
 </part>
 <part name="GND88" library="supply1" library_urn="urn:adsk.eagle:library:371" deviceset="GND" device=""/>
@@
 <part name="R24" library="rcl" deviceset="R-EU_" device="R0402" value="1k">
 <attribute name="DIGKEYPN" value="541-1.00KYCT-ND"/>
-<attribute name="MPN" value="CRCW04021K00FKED"/>
+<attribute name="MPN" value="CRCW04021K00FKEDHP"/>
 </part>
 <part name="R36" library="rcl" deviceset="R-EU_" device="R0402" value="330R">
@@
 <part name="R30" library="rcl" deviceset="R-EU_" device="R0402" value="1k">
 <attribute name="DIGKEYPN" value="541-1.00KYCT-ND"/>
-<attribute name="MPN" value="CRCW04021K00FKED"/>
+<attribute name="MPN" value="CRCW04021K00FKEDHP"/>
 </part>
 <part name="R44" library="rcl" deviceset="R-EU_" device="R0402" value="330R">
@@
 <part name="R25" library="rcl" deviceset="R-EU_" device="R0402" value="1k">
 <attribute name="DIGKEYPN" value="541-1.00KYCT-ND"/>
-<attribute name="MPN" value="CRCW04021K00FKED"/>
+<attribute name="MPN" value="CRCW04021K00FKEDHP"/>
 </part>
 <part name="R37" library="rcl" deviceset="R-EU_" device="R0402" value="330R">
@@
 <part name="R31" library="rcl" deviceset="R-EU_" device="R0402" value="1k">
 <attribute name="DIGKEYPN" value="541-1.00KYCT-ND"/>
-<attribute name="MPN" value="CRCW04021K00FKED"/>
+<attribute name="MPN" value="CRCW04021K00FKEDHP"/>
 </part>
 <part name="R45" library="rcl" deviceset="R-EU_" device="R0402" value="330R">
@@
 </part>
 <part name="R54" library="rcl" deviceset="R-EU_" device="R0402" value="10k">
-<attribute name="DIGKEYPN" value="541-3959-1-ND"/>
-<attribute name="MPN" value="CRCW040210K0FKED"/>
+<attribute name="DIGKEYPN" value="541-1.00KYCT-ND"/>
+<attribute name="MPN" value="CRCW04021K00FKEDHP"/>
 </part>
 <part name="GND70" library="supply1" deviceset="GND" device="">
@@
 </part>
 <part name="R55" library="rcl" deviceset="R-EU_" device="R0402" value="10k">
-<attribute name="DIGKEYPN" value="541-3959-1-ND"/>
-<attribute name="MPN" value="CRCW040210K0FKED"/>
+<attribute name="DIGKEYPN" value="541-1.00KYCT-ND"/>
+<attribute name="MPN" value="CRCW04021K00FKEDHP"/>
 </part>
 <part name="+3V29" library="supply1" library_urn="urn:adsk.eagle:library:371" deviceset="+3V3" device="">
@@
 </part>
 <part name="C29" library="rcl" deviceset="C-EU" device="C0402" value="330nF">
-<attribute name="DIGKEYPN" value="445-6899-2-ND"/>
-<attribute name="MPN" value="CGA2B3X7R1H104K050BB"/>
+<attribute name="DIGKEYPN" value="490-3263-1-ND"/>
+<attribute name="MPN" value="GRM155R61A334KE15D"/>
 </part>
 <part name="OSC1" library="harp timestamp generator" deviceset="OSCILLATOR" device="" value="OSCILLATOR">
@@
 </part>
 <part name="R6" library="rcl" deviceset="R-EU_" device="R0402" value="100k">
-<attribute name="DIGKEYPN" value="311-100KHRCT-ND"/>
-<attribute name="MPN" value="RC0603FR-07100KL"/>
+<attribute name="DIGKEYPN" value="P15984CT-ND"/>
+<attribute name="MPN" value="ERJ-2RHD1002X"/>
 </part>
 <part name="R7" library="rcl" deviceset="R-EU_" device="R0402" value="10k">
@@
 </part>
 <part name="R8" library="rcl" deviceset="R-EU_" device="R0402" value="0">
-<attribute name="DIGKEYPN" value="311-0.0HRCT-ND"/>
-<attribute name="MPN" value="RC0603FR-070RL"/>
+<attribute name="DIGKEYPN" value="RMCF0402ZT0R00CT-ND"/>
+<attribute name="MPN" value="RMCF0402ZT0R00"/>
 </part>
 <part name="GND41" library="supply1" deviceset="GND" device="">
@@
 </part>
 <part name="R48" library="rcl" deviceset="R-EU_" device="R0402" value="100k">
-<attribute name="DIGKEYPN" value="311-100KHRCT-ND"/>
-<attribute name="MPN" value="RC0603FR-07100KL"/>
+<attribute name="DIGKEYPN" value="P15984CT-ND"/>
+<attribute name="MPN" value="ERJ-2RHD1002X"/>
 </part>
 <part name="IC9" library="74xx-little-de" deviceset="74*1G126" device="DCK" technology="AHC" value="M74VHC1GT126DF1G">
